Commit message: Change the uri of meshes by  relative path

File: models/gr_robot/model_urdf.urdf (robot description, URDF)
Before this commit: robot gr_robot, 9 links, 8 joints
Links:
- link RS16_link: geometry collision cylinder length=0.08 radius=0.04; visual mesh filename=package://gr_description/models/gr_robot/meshes/accessories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 scale=0.001 0.001 0.001
- link base_link: geometry collision mesh filename=package://gr_description/models/gr_robot/meshes/accessories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 scale=0.001 0.001 0.001; collision mesh filename=package://gr_description/models/gr_robot/meshes/agilex/scou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 scale=1 1 1
- link camera_link: geometry collision box size=0.02505 0.09 0.025; visual mesh filename=package://gr_description/models/gr_robot/meshes/accessories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 scale=1 1 1
- link left_front_wheel_link: geometry collision mesh filename=package://gr_description/models/gr_robot/meshes/agilex/scou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 scale=1 1 1; visual mesh filename=package://gr_description/models/gr_robot/meshes/agilex/scou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 scale=1 1 1
- link left_rear_wheel_link: geometry collision mesh filename=package://gr_description/models/gr_robot/meshes/agilex/scou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 scale=1 1 1; visual mesh filename=package://gr_description/models/gr_robot/meshes/agilex/scou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 scale=1 1 1
- link right_front_wheel_link: geometry collision mesh filename=package://gr_description/models/gr_robot/meshes/agilex/scou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 scale=1 1 1; visual mesh filename=package://gr_description/models/gr_robot/meshes/agilex/scou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 scale=1 1 1
- link right_rear_wheel_link: geometry collision mesh filename=package://gr_description/models/gr_robot/meshes/agilex/scou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 scale=1 1 1; visual mesh filename=package://gr_description/models/gr_robot/meshes/agilex/scou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 scale=1 1 1
